File: wled-controller.sch (KiCad schematic (older format))
At the start: 37 parts

Commit message: First routing.
Parts:
- C1, C4: renamed from C?; footprint (none) -> Capacitor_THT:CP_Radial_D8.0mm_P3.50mm
- C2, C3, C5, C6, C7, C8: renamed from C?; footprint (none) -> Capacitor_SMD:C_0805_2012Metric_Pad1.18x1.45mm_HandSolder
- J1: renamed from J?; footprint (none) -> TerminalBlock_4Ucon:TerminalBlock_4Ucon_1x04_P3.50mm_Horizontal
- J2: renamed from J?; value Screw_Terminal_01x04 -> Screw_Terminal_01x06; footprint (none) -> TerminalBlock_4Ucon:TerminalBlock_4Ucon_1x06_P3.50mm_Horizontal; symbol Connector:Screw_Terminal_01x04 -> Connector:Screw_Terminal_01x06
- J3: renamed from J?; footprint (none) -> Connector_PinHeader_2.00mm:PinHeader_1x05_P2.00mm_Vertical
- R1, R2, R3, R4, R5, R6, R7, R8: renamed from R?; footprint (none) -> Resistor_SMD:R_0805_2012Metric_Pad1.20x1.40mm_HandSolder
- SW1: renamed from SW?; footprint (none) -> Button_Switch_THT:SW_PUSH_6mm_H13mm
- SW2: renamed from SW?; footprint (none) -> Button_Switch_THT:SW_PUSH_6mm_H8mm
- U1: renamed from U?; footprint (none) -> Package_TO_SOT_SMD:SOT-223-3_TabPin2
- U2: renamed from U?; footprint (none) -> Package_SO:SO-14_3.9x8.65mm_P1.27mm
- U3: renamed from U?; footprint RF_Module:ESP-07 -> wled-controller:ESP-07-tht
- gave numbers to parts that had none: 9
Connections:
- net +5V: now also J2.1 (Pin_1), J2.6 (Pin_6)
- net DATA_OUT: now also J2.5 (Pin_5); no longer J2.4 (Pin_4)
- net GND: now also J2.4 (Pin_4); no longer J2.2 (Pin_2)
- net SWITCH_IN: now also J2.2 (Pin_2); no longer J2.1 (Pin_1)
Other:
- note added: "FTDI Connector"
- moved on the sheet: C7, C8, J3, U4, U5

Commit message: V1.0
Parts:
- U3: footprint wled-controller:ESP-07-tht -> ESP8266:ESP-07_tht
Changed lines of the file:
@@
 F 0 "U3" H 5250 3300 50  0000 C CNN
 F 1 "ESP-07" H 5250 3200 50  0000 C CNN
-F 2 "wled-controller:ESP-07-tht" H 5550 2350 50  0001 C CNN
+F 2 "ESP8266:ESP-07_tht" H 5550 2350 50  0001 C CNN
 F 3 "http://wiki.ai-thinker.com/_media/esp8266/esp8266_series_modules_user_manual_v1.1.pdf" H 5200 2450 50  0001 C CNN
 	1    5550 2350

Commit message: Rev 2 with open Collector PS switch
Parts:
- added Q1: BC817, Package_TO_SOT_SMD:SOT-23, symbol Transistor_BJT:BC817
- added R10: 1k2, Resistor_SMD:R_0805_2012Metric_Pad1.20x1.40mm_HandSolder, symbol Device:R
- added R9: 10k, Resistor_SMD:R_0805_2012Metric_Pad1.20x1.40mm_HandSolder, symbol Device:R
- U3: footprint ESP8266:ESP-07_tht -> ESP8266:ESP-07v2
Connections:
- net GND: now also Q1.2 (E), R9.2
- net ESP_RELAY: no longer names the net of D3.2 (A), D6.1 (K), R7.1
- net ESP_RELAY: now also Q1.3 (C); no longer U3.6 (GPIO12)
- net RELAY_OUT renamed PS_ON
- new net: Q1.1 (B), R10.1
- new net ESP_PS_ON: R10.2, R9.1, U3.6 (GPIO12)
Changed lines of the file:
@@
 F 0 "U3" H 5250 3300 50  0000 C CNN
 F 1 "ESP-07" H 5250 3200 50  0000 C CNN
-F 2 "ESP8266:ESP-07_tht" H 5550 2350 50  0001 C CNN
+F 2 "ESP8266:ESP-07v2" H 5550 2350 50  0001 C CNN
 F 3 "http://wiki.ai-thinker.com/_media/esp8266/esp8266_series_modules_user_manual_v1.1.pdf" H 5200 2450 50  0001 C CNN
 	1    5550 2350
@@
 ESP_SW1
 Text GLabel 6700 2350 2    50   Input ~ 0
-ESP_RELAY
+ESP_PS_ON
 Wire Wire Line
 	6150 2150 6700 2150
@@
 	0    -1   1    0
 $EndComp
-Text GLabel 8950 2550 0    50   Output ~ 0
-ESP_RELAY
+Text GLabel 7800 2800 0    50   Output ~ 0
+ESP_PS_ON
 $Comp
 L Device:R R7
@@
 	-1   0    0    -1
 $EndComp
-Wire Wire Line
-	9450 2550 8950 2550
 Connection ~ 9450 2550
 NoConn ~ 4950 2150
@@
 $EndComp
 Text GLabel 1800 3500 2    50   Output ~ 0
-RELAY_OUT
+PS_ON
 Wire Wire Line
 	1400 3500 1800 3500
@@
 DATA_OUT
 Text GLabel 10250 2550 2    50   Input ~ 0
-RELAY_OUT
+PS_ON
 Text GLabel 10250 3650 2    50   Input ~ 0
 SWITCH_IN
@@
 Wire Wire Line
 	3400 3100 3650 3100
+$Comp
+L Transistor_BJT:BC817 Q1
+U 1 1 6164A9B5
+P 8750 2800
+F 0 "Q1" H 8941 2846 50  0000 L CNN
+F 1 "BC817" H 8941 2755 50  0000 L CNN
+F 2 "Package_TO_SOT_SMD:SOT-23" H 8950 2725 50  0001 L CIN
+F 3 "https://www.onsemi.com/pub/Collateral/BC818-D.pdf" H 8750 2800 50  0001 L CNN
+	1    8750 2800
+	1    0    0    -1
+$EndComp
+$Comp
+L Device:R R9
+U 1 1 61655DD1
+P 8000 3100
+F 0 "R9" H 8070 3146 50  0000 L CNN
+F 1 "10k" H 8070 3055 50  0000 L CNN
+F 2 "Resistor_SMD:R_0805_2012Metric_Pad1.20x1.40mm_HandSolder" V 7930 3100 50  0001 C CNN
+F 3 "~" H 8000 3100 50  0001 C CNN
+	1    8000 3100
+	1    0    0    -1
+$EndComp
+$Comp
+L Device:R R10
+U 1 1 61656A82
+P 8400 2800
+F 0 "R10" V 8193 2800 50  0000 C CNN
+F 1 "1k2" V 8284 2800 50  0000 C CNN
+F 2 "Resistor_SMD:R_0805_2012Metric_Pad1.20x1.40mm_HandSolder" V 8330 2800 50  0001 C CNN
+F 3 "~" H 8400 2800 50  0001 C CNN
+	1    8400 2800
+	0    1    1    0
+$EndComp
+Wire Wire Line
+	8850 2600 8850 2550
+Wire Wire Line
+	8850 2550 9450 2550
+Wire Wire Line
+	7800 2800 8000 2800
+Wire Wire Line
+	8000 2950 8000 2800
+Connection ~ 8000 2800
+Wire Wire Line
+	8000 2800 8250 2800
+$Comp
+L power:GND #PWR0138
+U 1 1 61671A25
+P 8000 3250
+F 0 "#PWR0138" H 8000 3000 50  0001 C CNN
+F 1 "GND" H 8005 3077 50  0000 C CNN
+F 2 "" H 8000 3250 50  0001 C CNN
+F 3 "" H 8000 3250 50  0001 C CNN
+	1    8000 3250
+	-1   0    0    -1
+$EndComp
+$Comp
+L power:GND #PWR0139
+U 1 1 61671E49
+P 8850 3000
+F 0 "#PWR0139" H 8850 2750 50  0001 C CNN
+F 1 "GND" H 8855 2827 50  0000 C CNN
+F 2 "" H 8850 3000 50  0001 C CNN
+F 3 "" H 8850 3000 50  0001 C CNN
+	1    8850 3000
+	-1   0    0    -1
+$EndComp
 $EndSCHEMATC

Commit message: Changed input diode to 1N5817.
Parts:
- removed D1: 1N4001, Diode_THT:D_DO-41_SOD81_P10.16mm_Horizontal, symbol Diode:1N4001
- added D1: 1N5817, Diode_THT:D_DO-41_SOD81_P10.16mm_Horizontal, symbol Diode:1N5817
Connections:
- net +5V: now also D1.1 (K)
- net at J1.4 (Pin_4): now also D1.2 (A)
Changed lines of the file:
@@
-	-1   0    0    1
-$EndComp
-$Comp
-L Diode:1N4001 D1
-U 1 1 61976AAF
-P 1900 3200
-F 0 "D1" H 1900 2983 50  0000 C CNN
-F 1 "1N4001" H 1900 3074 50  0000 C CNN
-F 2 "Diode_THT:D_DO-41_SOD81_P10.16mm_Horizontal" H 1900 3025 50  0001 C CNN
-F 3 "http://www.vishay.com/docs/88503/1n4001.pdf" H 1900 3200 50  0001 C CNN
-	1    1900 3200
 	-1   0    0    1
 $EndComp
@@
 	-1   0    0    -1
 $EndComp
+$Comp
+L Diode:1N5817 D1
+U 1 1 6166855F
+P 1900 3200
+F 0 "D1" H 1900 2983 50  0000 C CNN
+F 1 "1N5817" H 1900 3074 50  0000 C CNN
+F 2 "Diode_THT:D_DO-41_SOD81_P10.16mm_Horizontal" H 1900 3025 50  0001 C CNN
+F 3 "http://www.vishay.com/docs/88525/1n5817.pdf" H 1900 3200 50  0001 C CNN
+	1    1900 3200
+	-1   0    0    1
+$EndComp
 $EndSCHEMATC

Commit message: Changed programming header to 2.54mm
Parts:
- J3: footprint Connector_PinHeader_2.00mm:PinHeader_1x05_P2.00mm_Vertical -> Connector_PinHeader_2.54mm:PinHeader_1x05_P2.54mm_Vertical
- SW2: footprint Button_Switch_THT:SW_PUSH_6mm_H8mm -> Button_Switch_THT:SW_PUSH_6mm_H13mm
Changed lines of the file:
@@
 F 0 "SW2" H 10100 6335 50  0000 C CNN
 F 1 "SW_Push" H 10100 6244 50  0000 C CNN
-F 2 "Button_Switch_THT:SW_PUSH_6mm_H8mm" H 10100 6250 50  0001 C CNN
+F 2 "Button_Switch_THT:SW_PUSH_6mm_H13mm" H 10100 6250 50  0001 C CNN
 F 3 "~" H 10100 6250 50  0001 C CNN
 	1    10100 6050
@@
 F 0 "J3" H 5708 7481 50  0000 C CNN
 F 1 "Conn_01x05_Male" H 5708 7390 50  0000 C CNN
-F 2 "Connector_PinHeader_2.00mm:PinHeader_1x05_P2.00mm_Vertical" H 5600 7100 50  0001 C CNN
+F 2 "Connector_PinHeader_2.54mm:PinHeader_1x05_P2.54mm_Vertical" H 5600 7100 50  0001 C CNN
 F 3 "~" H 5600 7100 50  0001 C CNN
 	1    5600 7100
